File: PCB/keycab.kicad_pcb (KiCad board)
At the start: 2 copper layers, 97.6 x 64.4 mm, 23 parts, among them J1 Conn_01x04_Socket, SW1 RotaryEncoder_Switch, SW22 SW_Push, SW23 SW_Push, SW24 SW_Push, SW25 SW_Push, SW26 SW_Push, SW27 SW_Push, SW28 SW_Push, SW29 SW_Push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

Commit message: Add files via upload
Parts:
- moved J1 23.0 mm to (80.0, 50.0)
Routing:
- net Net-(J1-Pin_1): track 188.3 -> 208.7 mm, vias 0 -> 4
- net Net-(J1-Pin_2): track 9.14 -> 27.3 mm, vias 0 -> 2
- net Net-(J1-Pin_3): track 63.7 -> 71.7 mm
- net Net-(U1-PA11_A3_D3): track 69.1 -> 76.1 mm, vias 4 -> 6
- net Net-(J1-Pin_4): track 34.2 -> 30.7 mm
